File: Hardware/V3.sch (EAGLE design)
At the start: 21 parts

Commit message: New Example / New hardware version
Parts:
- removed ANALOG, HACKPORT, JP5, JP6: (no value), pinhead:PINHD-1X6
Connections:
- removed net N$17: ANALOG.2, U$1.A10
- removed net N$18: ANALOG.3, U$1.23/A9
- removed net N$19: ANALOG.4, U$1.22/A8
- removed net N$20: HACKPORT.1, U$1.0
- removed net N$21: HACKPORT.2, U$1.1
- removed net N$24: HACKPORT.5, U$1.11
- removed net N$25: HACKPORT.6, U$1.12
- removed net N$28: ANALOG.5, U$1.21/A7
- net GND: no longer JP5.1, JP5.2, JP5.3, JP5.4, JP5.5, JP5.6
- net N$10: now also KEYPAD.4, U$1.4; no longer KEYPAD.2, U$1.3
- net N$11: now also U$1.3; no longer U$1.4
- net N$12: now also KEYPAD.2, U$1.2; no longer KEYPAD.4, U$1.5
- net N$13: no longer KEYPAD.5
- net N$16: now also KEYPAD.1, U$1.1; no longer ANALOG.1, U$1.A11
- net N$22: no longer HACKPORT.3
- net N$23: no longer HACKPORT.4
- net N$29: no longer ANALOG.6
- net N$7: now also KEYPAD.5, U$1.5; no longer KEYPAD.1, U$1.2
- net N$8: no longer JP6.1, JP6.2, JP6.3, JP6.4, JP6.5, JP6.6
