File: Hardware/V4.brd (EAGLE design)
At the start: 100 x 80 mm, 17 parts

Commit message: Hardware update / MIDI Sample updates
Parts:
- moved R12 21.1 mm to (34.3, 33.0)
- moved R8 21.1 mm to (29.2, 33.0)
- moved R10 21.1 mm to (24.1, 33.0)
- moved R9 21.1 mm to (19.1, 33.0)
- moved R11 20.1 mm to (39.4, 33.0)
- moved JP1 18.9 mm to (22.9, 74.9)
- moved C2 18.9 mm to (12.7, 62.2)
- moved KEYPAD 18.9 mm to (22.9, 61.0)
- moved R13 18.9 mm to (17.8, 55.9)
- moved U$1 18.9 mm to (35.6, 59.7)
- moved U$2 18.9 mm to (8.89, 68.6)
- moved R1 16.5 mm to (53.3, 8.89)
- moved R6 16.5 mm to (53.3, 72.4)
- moved R2 15.7 mm to (53.3, 21.6)
- moved R5 15.7 mm to (53.3, 59.7)
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Routing:
- net N$8: track 139.9 -> 204.6 mm
- net N$1: track 29.3 -> 45.3 mm
- net N$2: track 22.1 -> 34.2 mm
- net N$3: track 15.5 -> 25.7 mm
- net N$4: track 8.21 -> 13.3 mm
- net N$22: track 20.2 -> 15.1 mm
- net N$13: track 24.7 -> 19.6 mm
- net N$23: track 15.5 -> 10.5 mm
- net N$29: track 28.8 -> 24.7 mm
- net GND: track 3.81 -> 0.00 mm
- net N$26: track 11.5 -> 10.2 mm
- net N$6: track 20.2 -> 21.3 mm
